File: electrical/Balancing_robot_remote/remote.sch (KiCad schematic (older format))
At the start: 4 parts, among them U1 WRL-00691, U2 nunchuck

Commit message: added nunchuck wire colors
Other:
- note added: "Green wire"
- note added: "Red wire"
- note added: "White wire"
- note added: "Yellow wire"
Changed lines of the file:
@@
 	1    0    0    -1
 $EndComp
+Text Notes 9625 3670 0    50   ~ 0
+Yellow wire
+Text Notes 9625 3810 0    50   ~ 0
+White wire
+Text Notes 9630 3975 0    50   ~ 0
+Red wire
+Text Notes 9630 4135 0    50   ~ 0
+Green wire
 $EndSCHEMATC

Commit message: tweeked the schematic
Other:
- moved on the sheet: U2
Changed lines of the file:
@@
 EELAYER 25 0
 EELAYER END
-$Descr A4 11693 8268
+$Descr A 11000 8500
 encoding utf-8
 Sheet 1 1
@@
 Wire Wire Line
 	3300 3715 3245 3715
-Text Label 9095 3785 2    60   ~ 0
+Text Label 8235 4155 2    60   ~ 0
 SCL
-Text Label 9095 3645 2    60   ~ 0
+Text Label 8235 4015 2    60   ~ 0
 SDA
 Text Label 4295 4745 2    60   ~ 0
@@
 L nunchuck U2
 U 1 1 597F71F2
-P 9465 3865
-F 0 "U2" H 9465 3385 60  0000 C CNN
-F 1 "nunchuck" H 9455 4365 60  0000 C CNN
-F 2 "" H 9465 3865 60  0001 C CNN
-F 3 "" H 9465 3865 60  0001 C CNN
-	1    9465 3865
+P 8605 4235
+F 0 "U2" H 8605 3755 60  0000 C CNN
+F 1 "nunchuck" H 8595 4735 60  0000 C CNN
+F 2 "" H 8605 4235 60  0001 C CNN
+F 3 "" H 8605 4235 60  0001 C CNN
+	1    8605 4235
 	1    0    0    -1
 $EndComp
@@
 L GND #PWR9
 U 1 1 597F7363
-P 8805 3945
-F 0 "#PWR9" H 8805 3695 50  0001 C CNN
-F 1 "GND" H 8805 3795 50  0000 C CNN
-F 2 "" H 8805 3945 50  0000 C CNN
-F 3 "" H 8805 3945 50  0000 C CNN
-	1    8805 3945
-	1    0    0    -1
-$EndComp
-Wire Wire Line
-	9095 3945 8805 3945
-Wire Wire Line
-	9095 4105 9095 4165
-Wire Wire Line
-	9095 4165 8525 4165
+P 7945 4315
+F 0 "#PWR9" H 7945 4065 50  0001 C CNN
+F 1 "GND" H 7945 4165 50  0000 C CNN
+F 2 "" H 7945 4315 50  0000 C CNN
+F 3 "" H 7945 4315 50  0000 C CNN
+	1    7945 4315
+	1    0    0    -1
+$EndComp
+Wire Wire Line
+	8235 4315 7945 4315
+Wire Wire Line
+	8235 4475 8235 4535
+Wire Wire Line
+	8235 4535 7665 4535
 $Comp
 L +3.3V #PWR6
@@
 L +3.3V #PWR8
 U 1 1 597F771C
-P 8525 4165
-F 0 "#PWR8" H 8525 4015 50  0001 C CNN
-F 1 "+3.3V" H 8525 4305 50  0000 C CNN
-F 2 "" H 8525 4165 50  0000 C CNN
-F 3 "" H 8525 4165 50  0000 C CNN
-	1    8525 4165
-	1    0    0    -1
-$EndComp
-Text Notes 9625 3670 0    50   ~ 0
+P 7665 4535
+F 0 "#PWR8" H 7665 4385 50  0001 C CNN
+F 1 "+3.3V" H 7665 4675 50  0000 C CNN
+F 2 "" H 7665 4535 50  0000 C CNN
+F 3 "" H 7665 4535 50  0000 C CNN
+	1    7665 4535
+	1    0    0    -1
+$EndComp
+Text Notes 8765 4040 0    50   ~ 0
 Yellow wire
-Text Notes 9625 3810 0    50   ~ 0
+Text Notes 8765 4180 0    50   ~ 0
 White wire
-Text Notes 9630 3975 0    50   ~ 0
+Text Notes 8770 4345 0    50   ~ 0
 Red wire
-Text Notes 9630 4135 0    50   ~ 0
+Text Notes 8770 4505 0    50   ~ 0
 Green wire
 $EndSCHEMATC

Commit message: working on the firmware tests
Other:
- moved on the sheet: U2
Changed lines of the file:
@@
 Wire Wire Line
 	3300 3715 3245 3715
-Text Label 8235 4155 2    60   ~ 0
+Text Label 7425 4275 2    60   ~ 0
 SCL
-Text Label 8235 4015 2    60   ~ 0
+Text Label 7425 4135 2    60   ~ 0
 SDA
 Text Label 4295 4745 2    60   ~ 0
@@
 L nunchuck U2
 U 1 1 597F71F2
-P 8605 4235
-F 0 "U2" H 8605 3755 60  0000 C CNN
-F 1 "nunchuck" H 8595 4735 60  0000 C CNN
-F 2 "" H 8605 4235 60  0001 C CNN
-F 3 "" H 8605 4235 60  0001 C CNN
-	1    8605 4235
+P 7795 4355
+F 0 "U2" H 7795 3875 60  0000 C CNN
+F 1 "nunchuck" H 7785 4855 60  0000 C CNN
+F 2 "" H 7795 4355 60  0001 C CNN
+F 3 "" H 7795 4355 60  0001 C CNN
+	1    7795 4355
 	1    0    0    -1
 $EndComp
@@
 L GND #PWR9
 U 1 1 597F7363
-P 7945 4315
-F 0 "#PWR9" H 7945 4065 50  0001 C CNN
-F 1 "GND" H 7945 4165 50  0000 C CNN
-F 2 "" H 7945 4315 50  0000 C CNN
-F 3 "" H 7945 4315 50  0000 C CNN
-	1    7945 4315
+P 7135 4435
+F 0 "#PWR9" H 7135 4185 50  0001 C CNN
+F 1 "GND" H 7135 4285 50  0000 C CNN
+F 2 "" H 7135 4435 50  0000 C CNN
+F 3 "" H 7135 4435 50  0000 C CNN
+	1    7135 4435
 	1    0    0    -1
 $EndComp
 Wire Wire Line
-	8235 4315 7945 4315
+	7425 4435 7135 4435
 Wire Wire Line
-	8235 4475 8235 4535
+	7425 4595 7425 4655
 Wire Wire Line
-	8235 4535 7665 4535
+	7425 4655 6855 4655
 $Comp
 L +3.3V #PWR6
@@
 L +3.3V #PWR8
 U 1 1 597F771C
-P 7665 4535
-F 0 "#PWR8" H 7665 4385 50  0001 C CNN
-F 1 "+3.3V" H 7665 4675 50  0000 C CNN
-F 2 "" H 7665 4535 50  0000 C CNN
-F 3 "" H 7665 4535 50  0000 C CNN
-	1    7665 4535
+P 6855 4655
+F 0 "#PWR8" H 6855 4505 50  0001 C CNN
+F 1 "+3.3V" H 6855 4795 50  0000 C CNN
+F 2 "" H 6855 4655 50  0000 C CNN
+F 3 "" H 6855 4655 50  0000 C CNN
+	1    6855 4655
 	1    0    0    -1
 $EndComp
-Text Notes 8765 4040 0    50   ~ 0
+Text Notes 7955 4160 0    50   ~ 0
 Yellow wire
-Text Notes 8765 4180 0    50   ~ 0
+Text Notes 7955 4300 0    50   ~ 0
 White wire
-Text Notes 8770 4345 0    50   ~ 0
+Text Notes 7960 4465 0    50   ~ 0
 Red wire
-Text Notes 8770 4505 0    50   ~ 0
+Text Notes 7960 4625 0    50   ~ 0
 Green wire
 $EndSCHEMATC

Commit message: modified schematics to connect radio CE pin to pin D9 on the arduinos
Parts:
- removed R1: 0R, Resistors_SMD:R_0805_HandSoldering, symbol R_Small
Connections:
- net CE: now reaches U1.2 (CE)
- net CE: now also SHIELD1.9
- no-connect marks 18 -> 17
Changed lines of the file:
@@
 Text Notes 1970 3460 0    60   ~ 0
 SPI 2.5 GHz Wireless
-$Comp
-L +5V #PWR3
-U 1 1 5955B40F
-P 3300 3625
-F 0 "#PWR3" H 3300 3475 50  0001 C CNN
-F 1 "+5V" H 3300 3765 50  0000 C CNN
-F 2 "" H 3300 3625 50  0000 C CNN
-F 3 "" H 3300 3625 50  0000 C CNN
-	1    3300 3625
-	1    0    0    -1
-$EndComp
-$Comp
-L R_Small R1
-U 1 1 5955CF79
-P 3145 3715
-F 0 "R1" H 3175 3735 50  0000 L CNN
-F 1 "0R" H 3175 3675 50  0000 L CNN
-F 2 "Resistors_SMD:R_0805_HandSoldering" H 3145 3715 50  0001 C CNN
-F 3 "" H 3145 3715 50  0000 C CNN
-F 4 "Value" H 3145 3715 60  0001 C CNN "Fieldname"
-	1    3145 3715
-	0    -1   -1   0
-$EndComp
 Wire Wire Line
 	1845 3990 1845 3915
@@
 Wire Wire Line
 	1835 3755 1935 3755
-Wire Wire Line
-	3045 3715 2975 3715
-Wire Wire Line
-	3300 3625 3300 3715
-Wire Wire Line
-	3300 3715 3245 3715
 Text Label 7425 4275 2    60   ~ 0
 SCL
@@
 	1    0    0    -1
 $EndComp
-NoConn ~ 6195 3745
 NoConn ~ 6195 3845
 NoConn ~ 6195 4045
@@
 Text Notes 7960 4625 0    50   ~ 0
 Green wire
+Text Label 6195 3745 0    60   ~ 0
+CE
+Text Label 2975 3715 0    60   ~ 0
+CE
 $EndSCHEMATC
