File: electrical/Balancing_robot/balancingBot.sch (KiCad schematic (older format))
At the start: 33 parts, among them P1 CONN_01X02, P2 CONN_01X02, P3 CONN_01X02, P4 CONN_01X02, P5 CONN_01X02, P6 CONN_01X02, SW1 SW_DIP_x01, U1 DRV8825, U2 DRV8825, U3 WRL-00691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

Commit message: tweeked the schematic
Parts:
- removed P1, P2, P4, P5: CONN_01X02, Socket_Strips:Socket_Strip_Straight_1x02, symbol CONN_01X02
- removed R1, R10, R13, R14, R2, R4, R7, R8: NOPOP, Resistors_SMD:R_0805_HandSoldering, symbol R_Small
- removed R11, R12, R15, R3, R5, R6, R9: 0R, Resistors_SMD:R_0805_HandSoldering, symbol R_Small
- added P? (x2): CONN_01X04, symbol CONN_01X04
Connections:
- net labels added: 11.75V
- net labels removed: 11.1V
- wire segments 138 -> 96
- no-connect marks 30 -> 35
Other:
- note added: "Voltages:\nMaximum 3S Lipo voltage = 12.6V.\nNominal 3S Lipo voltage = 11.1V.\nSafe drain 3S Lipo voltage = 9.9V.\nNo current diode drop = 0.512V.\nFull current diode drop = 0.83V to 0.87V.\nTherefore, max supply voltage = 11.73V to 12.09V.\nNominal supply voltage = 10.23V to 10.59V.\nMin safe supply voltage = 9.03V to 9.39V."
- moved on the sheet: D1, P3, P6, U5, U6

Commit message: converted to pcb and initial pcb layout
Parts:
- removed P6: CONN_01X02, Socket_Strips:Socket_Strip_Straight_1x02, symbol CONN_01X02
- removed SW1: SW_DIP_x01, Buttons_Switches_THT:SW_DIP_x1_Slide, symbol SW_DIP_x01
- added R103, R105, R106, R108: NOPOP, Resistors_SMD:R_0805_HandSoldering, symbol R_Small
- added R104, R107: 0R, Resistors_SMD:R_0805_HandSoldering, symbol R_Small
- added SW101: SW_SPDT, balancingBot:SWITCH-200MSP1T1B1M2QEH, symbol SW_SPDT
- C101: renamed from C1; footprint (none) -> Capacitors_THT:C_Radial_D7.5_L11.2_P2.5
- C102: renamed from C2; footprint (none) -> Capacitors_THT:C_Radial_D7.5_L11.2_P2.5
- D101: renamed from D1; footprint balancingBot:TMiniP2-F2-B -> Diodes_THT:Diode_DO-41_SOD81_Horizontal_RM10
- P101, P102: renamed from P?; footprint (none) -> Pin_Headers:Pin_Header_Straight_1x04
- P103: renamed from P3; footprint Socket_Strips:Socket_Strip_Straight_1x02 -> balancingBot:Terminal_Block_200_mil
- R101: renamed from R16; value 3K3 -> 33K
- R102: renamed from R17; value 2K2 -> 21K5
- renumbered U3 to U101, U2 to U102, U1 to U103, U4 to U104, U6 to U105, U5 to U106
Connections:
- wire segments 96 -> 110
- no-connect marks 35 -> 26

Commit message: working on the firmware tests
Connections:
- net Ldir: now also U103.9 (DIR), U104.8 (D5); no longer U102.9 (DIR), U104.6 (D3)
- net Lstep: now also U103.10 (STEP), U104.7 (D4); no longer U102.10 (STEP), U104.5 (D2)
- net Rdir: now also U102.9 (DIR), U104.6 (D3); no longer U103.9 (DIR), U104.8 (D5)
- net Rstep: now also U102.10 (STEP), U104.5 (D2); no longer U103.10 (STEP), U104.7 (D4)
Other:
- note added: "Blue\nRed\nBlack\nGreen"
- note added: "Green\nBlack\nRed\nBlue"
Changed lines of the file:
@@
 	1    0    0    -1
 $EndComp
-Text Notes 2435 4320 0    60   ~ 0
+Text Notes 2370 6430 0    60   ~ 0
 Right Stepper
-Text Notes 2390 6465 0    60   ~ 0
+Text Notes 2435 4295 0    60   ~ 0
 Left Stepper
 Text Notes 9285 5290 0    60   ~ 0
@@
 Text Notes 5360 1635 0    60   ~ 0
 Voltage Sense
+Text Label 2795 1695 2    60   ~ 0
+Rstep
+Text Label 2795 1795 2    60   ~ 0
+Rdir
+Text Label 2205 7250 2    50   ~ 0
+Rdir
+Text Label 2795 1965 2    60   ~ 0
+Ldir
 Text Label 2795 1885 2    60   ~ 0
-Rstep
-Text Label 2795 1965 2    60   ~ 0
-Rdir
-Text Label 2240 5105 2    50   ~ 0
-Rdir
-Text Label 2795 1795 2    60   ~ 0
-Ldir
-Text Label 2795 1695 2    60   ~ 0
 Lstep
 Text Label 9025 5585 2    60   ~ 0
@@
 NoConn ~ 2240 4585
 NoConn ~ 3160 5035
-Text Label 2205 7180 2    50   ~ 0
+Text Label 2240 5035 2    50   ~ 0
 Lstep
-Text Label 2205 7250 2    50   ~ 0
+Text Label 2240 5105 2    50   ~ 0
 Ldir
 NoConn ~ 2205 6730
@@
 	8270 3860 8270 3960
 NoConn ~ 8070 4060
-Text Label 2240 5035 2    50   ~ 0
+Text Label 2205 7180 2    50   ~ 0
 Rstep
 $Comp
@@
 	1790 6540 1790 6505
 Connection ~ 1790 6505
+Text Notes 4655 5035 0    60   ~ 0
+Blue\nRed\nBlack\nGreen
+Text Notes 4370 7170 0    60   ~ 0
+Green\nBlack\nRed\nBlue
 $EndSCHEMATC

Commit message: finally,delayed update with a working bot
Parts:
- added D102: Red LED, symbol LED_Small
- added R109: 330R, symbol R_Small
Connections:
- net GND: now also R109.2
- net at U104.20 (A3/D17): now also D102.2 (A)
- new net: D102.1 (K), R109.1
- no-connect marks 26 -> 25
Other:
- moved on the sheet: R101, R102
Changed lines of the file:
@@
 NoConn ~ 4105 1855
 NoConn ~ 4105 1765
-NoConn ~ 4105 1665
-$Comp
-L GND #PWR116
+$Comp
+L GND #PWR01
 U 1 1 59559CE8
 P 9975 6160
-F 0 "#PWR116" H 9975 5910 50  0001 C CNN
+F 0 "#PWR01" H 9975 5910 50  0001 C CNN
 F 1 "GND" H 9975 6010 50  0000 C CNN
 F 2 "" H 9975 6160 50  0000 C CNN
@@
 $EndComp
 $Comp
-L +5V #PWR115
+L +5V #PWR02
 U 1 1 59559D4A
 P 9975 5700
-F 0 "#PWR115" H 9975 5550 50  0001 C CNN
+F 0 "#PWR02" H 9975 5550 50  0001 C CNN
 F 1 "+5V" H 9975 5840 50  0000 C CNN
 F 2 "" H 9975 5700 50  0000 C CNN
@@
 11.75V
 $Comp
-L GND #PWR114
+L GND #PWR03
 U 1 1 5955A15B
 P 8390 4540
-F 0 "#PWR114" H 8390 4290 50  0001 C CNN
+F 0 "#PWR03" H 8390 4290 50  0001 C CNN
 F 1 "GND" H 8390 4390 50  0000 C CNN
 F 2 "" H 8390 4540 50  0000 C CNN
@@
 $EndComp
 $Comp
-L +5V #PWR117
+L +5V #PWR04
 U 1 1 5955A1EF
 P 10055 4270
-F 0 "#PWR117" H 10055 4120 50  0001 C CNN
+F 0 "#PWR04" H 10055 4120 50  0001 C CNN
 F 1 "+5V" H 10055 4410 50  0000 C CNN
 F 2 "" H 10055 4270 50  0000 C CNN
@@
 NoConn ~ 9810 4020
 $Comp
-L +5V #PWR101
+L +5V #PWR05
 U 1 1 5955A687
 P 710 1510
-F 0 "#PWR101" H 710 1360 50  0001 C CNN
+F 0 "#PWR05" H 710 1360 50  0001 C CNN
 F 1 "+5V" H 710 1650 50  0000 C CNN
 F 2 "" H 710 1510 50  0000 C CNN
@@
 $EndComp
 $Comp
-L GND #PWR102
+L GND #PWR06
 U 1 1 5955A6E0
 P 720 1790
-F 0 "#PWR102" H 720 1540 50  0001 C CNN
+F 0 "#PWR06" H 720 1540 50  0001 C CNN
 F 1 "GND" H 720 1640 50  0000 C CNN
 F 2 "" H 720 1790 50  0000 C CNN
@@
 5V 1A
 $Comp
-L +5V #PWR105
+L +5V #PWR07
 U 1 1 5955B40F
 P 2175 1425
-F 0 "#PWR105" H 2175 1275 50  0001 C CNN
+F 0 "#PWR07" H 2175 1275 50  0001 C CNN
 F 1 "+5V" H 2175 1565 50  0000 C CNN
 F 2 "" H 2175 1425 50  0000 C CNN
@@
 11.75V
 $Comp
-L GND #PWR110
+L GND #PWR08
 U 1 1 5955B554
 P 3770 4430
-F 0 "#PWR110" H 3770 4180 50  0001 C CNN
+F 0 "#PWR08" H 3770 4180 50  0001 C CNN
 F 1 "GND" H 3770 4280 50  0000 C CNN
 F 2 "" H 3770 4430 50  0000 C CNN
@@
 $EndComp
 $Comp
-L GND #PWR108
+L GND #PWR09
 U 1 1 5955B696
 P 3160 5210
-F 0 "#PWR108" H 3160 4960 50  0001 C CNN
+F 0 "#PWR09" H 3160 4960 50  0001 C CNN
 F 1 "GND" H 3160 5060 50  0000 C CNN
 F 2 "" H 3160 5210 50  0000 C CNN
@@
 11.75V
 $Comp
-L GND #PWR109
+L GND #PWR010
 U 1 1 5955B883
 P 3735 6575
-F 0 "#PWR109" H 3735 6325 50  0001 C CNN
+F 0 "#PWR010" H 3735 6325 50  0001 C CNN
 F 1 "GND" H 3735 6425 50  0000 C CNN
 F 2 "" H 3735 6575 50  0000 C CNN
@@
 $EndComp
 $Comp
-L GND #PWR107
+L GND #PWR011
 U 1 1 5955BA2D
 P 3125 7355
-F 0 "#PWR107" H 3125 7105 50  0001 C CNN
+F 0 "#PWR011" H 3125 7105 50  0001 C CNN
 F 1 "GND" H 3125 7205 50  0000 C CNN
 F 2 "" H 3125 7355 50  0000 C CNN
@@
 M0/M1/M2:\n0 0 0 - Full Step\n1 0 0 - 1/2 Step\n0 1 0 - 1/4 Step\n1 1 0 - 1/8 Step\n0 0 1 - 1/16 Step\nInternal pull down\n
 $Comp
-L +5V #PWR104
+L +5V #PWR012
 U 1 1 59569A5C
 P 1485 4345
-F 0 "#PWR104" H 1485 4195 50  0001 C CNN
+F 0 "#PWR012" H 1485 4195 50  0001 C CNN
 F 1 "+5V" H 1485 4485 50  0000 C CNN
 F 2 "" H 1485 4345 50  0000 C CNN
@@
 L R_Small R101
 U 1 1 595697E0
-P 5195 1470
-F 0 "R101" H 5225 1490 50  0000 L CNN
-F 1 "33K" H 5225 1430 50  0000 L CNN
-F 2 "Resistors_SMD:R_0805_HandSoldering" H 5195 1470 50  0001 C CNN
-F 3 "" H 5195 1470 50  0000 C CNN
-F 4 "Value" H 5195 1470 60  0001 C CNN "Fieldname"
-	1    5195 1470
+P 5585 1680
+F 0 "R101" H 5615 1700 50  0000 L CNN
+F 1 "33K" H 5615 1640 50  0000 L CNN
+F 2 "Resistors_SMD:R_0805_HandSoldering" H 5585 1680 50  0001 C CNN
+F 3 "" H 5585 1680 50  0000 C CNN
+F 4 "Value" H 5585 1680 60  0001 C CNN "Fieldname"
+	1    5585 1680
 	1    0    0    -1
 $EndComp
@@
 L R_Small R102
 U 1 1 5956988A
-P 5195 1735
-F 0 "R102" H 5225 1755 50  0000 L CNN
-F 1 "21K5" H 5225 1695 50  0000 L CNN
-F 2 "Resistors_SMD:R_0805_HandSoldering" H 5195 1735 50  0001 C CNN
-F 3 "" H 5195 1735 50  0000 C CNN
-F 4 "Value" H 5195 1735 60  0001 C CNN "Fieldname"
-	1    5195 1735
-	1    0    0    -1
-$EndComp
-$Comp
-L GND #PWR113
+P 5585 1945
+F 0 "R102" H 5615 1965 50  0000 L CNN
+F 1 "21K5" H 5615 1905 50  0000 L CNN
+F 2 "Resistors_SMD:R_0805_HandSoldering" H 5585 1945 50  0001 C CNN
+F 3 "" H 5585 1945 50  0000 C CNN
+F 4 "Value" H 5585 1945 60  0001 C CNN "Fieldname"
+	1    5585 1945
+	1    0    0    -1
+$EndComp
+$Comp
+L GND #PWR013
 U 1 1 59569A75
-P 5195 1885
-F 0 "#PWR113" H 5195 1635 50  0001 C CNN
-F 1 "GND" H 5195 1735 50  0000 C CNN
-F 2 "" H 5195 1885 50  0000 C CNN
-F 3 "" H 5195 1885 50  0000 C CNN
-	1    5195 1885
-	1    0    0    -1
-$EndComp
-Text GLabel 5300 1180 2    60   Input ~ 0
+P 5585 2095
+F 0 "#PWR013" H 5585 1845 50  0001 C CNN
+F 1 "GND" H 5585 1945 50  0000 C CNN
+F 2 "" H 5585 2095 50  0000 C CNN
+F 3 "" H 5585 2095 50  0000 C CNN
+	1    5585 2095
+	1    0    0    -1
+$EndComp
+Text GLabel 5690 1390 2    60   Input ~ 0
 11.75V
-Text Notes 5360 1635 0    60   ~ 0
+Text Notes 5750 1845 0    60   ~ 0
 Voltage Sense
 Text Label 2795 1695 2    60   ~ 0
@@
 NoConn ~ 3125 7180
 $Comp
-L GND #PWR111
+L GND #PWR014
 U 1 1 59AC80BA
 P 4270 1110
-F 0 "#PWR111" H 4270 860 50  0001 C CNN
+F 0 "#PWR014" H 4270 860 50  0001 C CNN
 F 1 "GND" H 4270 960 50  0000 C CNN
 F 2 "" H 4270 1110 50  0000 C CNN
@@
 $EndComp
 $Comp
-L +5V #PWR112
+L +5V #PWR015
 U 1 1 59AC8320
 P 4470 1470
-F 0 "#PWR112" H 4470 1320 50  0001 C CNN
+F 0 "#PWR015" H 4470 1320 50  0001 C CNN
 F 1 "+5V" H 4470 1610 50  0000 C CNN
 F 2 "" H 4470 1470 50  0000 C CNN
@@
 $EndComp
 $Comp
-L GND #PWR106
+L GND #PWR016
 U 1 1 59AC848A
 P 2370 1665
-F 0 "#PWR106" H 2370 1415 50  0001 C CNN
+F 0 "#PWR016" H 2370 1415 50  0001 C CNN
 F 1 "GND" H 2370 1515 50  0000 C CNN
 F 2 "" H 2370 1665 50  0000 C CNN
@@
 Connection ~ 8390 4240
 Wire Wire Line
-	5300 1180 5195 1180
-Wire Wire Line
-	5195 1180 5195 1370
-Wire Wire Line
-	5195 1570 5195 1635
-Wire Wire Line
-	5195 1835 5195 1885
+	5690 1390 5585 1390
+Wire Wire Line
+	5585 1390 5585 1580
+Wire Wire Line
+	5585 1780 5585 1845
+Wire Wire Line
+	5585 2045 5585 2095
 Wire Wire Line
 	4105 1935 4335 1935
 Wire Wire Line
-	4335 1935 4335 1605
-Wire Wire Line
-	4335 1605 5195 1605
-Connection ~ 5195 1605
+	4335 1815 5585 1815
+Connection ~ 5585 1815
 Wire Wire Line
 	3120 6200 3120 6210
@@
 Connection ~ 1825 4360
 $Comp
-L +5V #PWR103
+L +5V #PWR017
 U 1 1 59ADD131
 P 1450 6490
-F 0 "#PWR103" H 1450 6340 50  0001 C CNN
+F 0 "#PWR017" H 1450 6340 50  0001 C CNN
 F 1 "+5V" H 1450 6630 50  0000 C CNN
 F 2 "" H 1450 6490 50  0000 C CNN
@@
 Text Notes 4370 7170 0    60   ~ 0
 Green\nBlack\nRed\nBlue
+Wire Wire Line
+	4335 1935 4335 1815
+$Comp
+L R_Small R109
+U 1 1 5A80AAAD
+P 5005 1385
+F 0 "R109" H 5035 1405 50  0000 L CNN
+F 1 "330R" H 5035 1345 50  0000 L CNN
+F 2 "" H 5005 1385 50  0000 C CNN
+F 3 "" H 5005 1385 50  0000 C CNN
+F 4 "Value" H 5005 1385 60  0001 C CNN "Fieldname"
+	1    5005 1385
+	1    0    0    -1
+$EndComp
+$Comp
+L LED_Small D102
+U 1 1 5A80AB29
+P 5005 1035
+F 0 "D102" H 4955 1160 50  0000 L CNN
+F 1 "Red LED" H 4830 935 50  0000 L CNN
+F 2 "" V 5005 1035 50  0000 C CNN
+F 3 "" V 5005 1035 50  0000 C CNN
+F 4 "Value" H 5005 1035 60  0001 C CNN "Fieldname"
+	1    5005 1035
+	0    -1   -1   0
+$EndComp
+$Comp
+L GND #PWR018
+U 1 1 5A80ACDE
+P 5005 1545
+F 0 "#PWR018" H 5005 1295 50  0001 C CNN
+F 1 "GND" H 5005 1395 50  0000 C CNN
+F 2 "" H 5005 1545 50  0000 C CNN
+F 3 "" H 5005 1545 50  0000 C CNN
+	1    5005 1545
+	1    0    0    -1
+$EndComp
+Wire Wire Line
+	5005 1485 5005 1545
+Wire Wire Line
+	5005 1135 5005 1285
+Wire Wire Line
+	4105 1665 4665 1665
+Wire Wire Line
+	4665 1665 4665 935
+Wire Wire Line
+	4665 935  5005 935
 $EndSCHEMATC

Commit message: modified schematics to connect radio CE pin to pin D9 on the arduinos
Connections:
- net +5V: no longer U101.2 (CE)
- net CE: now reaches U104.12 (D9)
- net CE: now also U101.2 (CE)
- no-connect marks 25 -> 24
Changed lines of the file:
@@
 Text Notes 9245 3615 0    60   ~ 0
 5V 1A
-$Comp
-L +5V #PWR07
-U 1 1 5955B40F
-P 2175 1425
-F 0 "#PWR07" H 2175 1275 50  0001 C CNN
-F 1 "+5V" H 2175 1565 50  0000 C CNN
-F 2 "" H 2175 1425 50  0000 C CNN
-F 3 "" H 2175 1425 50  0000 C CNN
-	1    2175 1425
-	1    0    0    -1
-$EndComp
 Text GLabel 3880 3640 2    60   Input ~ 0
 11.75V
@@
 MISO
 NoConn ~ 2795 2225
-NoConn ~ 2795 2315
 Text Label 1850 1625 0    60   ~ 0
 CSN
@@
 	3125 7250 3125 7355
 Wire Wire Line
-	1850 1515 2175 1515
-Wire Wire Line
-	2175 1515 2175 1425
-Wire Wire Line
 	3125 6870 3905 6870
 Wire Wire Line
@@
 Wire Wire Line
 	4665 935  5005 935
+Text Label 2795 2315 2    60   ~ 0
+CE
+Text Label 1850 1515 0    60   ~ 0
+CE
 $EndSCHEMATC

Commit message: updated pcb to include status LED, associated resistor, and radio enable line
Parts:
- D102: footprint (none) -> LEDs:LED_0805_HandSoldering
- R109: footprint (none) -> Resistors_SMD:R_0805_HandSoldering
Other:
- note removed: "Blue\nRed\nBlack\nGreen"
Changed lines of the file:
@@
 11.75V
 $Comp
-L GND #PWR08
+L GND #PWR07
 U 1 1 5955B554
 P 3770 4430
-F 0 "#PWR08" H 3770 4180 50  0001 C CNN
+F 0 "#PWR07" H 3770 4180 50  0001 C CNN
 F 1 "GND" H 3770 4280 50  0000 C CNN
 F 2 "" H 3770 4430 50  0000 C CNN
@@
 $EndComp
 $Comp
-L GND #PWR09
+L GND #PWR08
 U 1 1 5955B696
 P 3160 5210
-F 0 "#PWR09" H 3160 4960 50  0001 C CNN
+F 0 "#PWR08" H 3160 4960 50  0001 C CNN
 F 1 "GND" H 3160 5060 50  0000 C CNN
 F 2 "" H 3160 5210 50  0000 C CNN
@@
 11.75V
 $Comp
-L GND #PWR010
+L GND #PWR09
 U 1 1 5955B883
 P 3735 6575
-F 0 "#PWR010" H 3735 6325 50  0001 C CNN
+F 0 "#PWR09" H 3735 6325 50  0001 C CNN
 F 1 "GND" H 3735 6425 50  0000 C CNN
 F 2 "" H 3735 6575 50  0000 C CNN
@@
 $EndComp
 $Comp
-L GND #PWR011
+L GND #PWR010
 U 1 1 5955BA2D
 P 3125 7355
-F 0 "#PWR011" H 3125 7105 50  0001 C CNN
+F 0 "#PWR010" H 3125 7105 50  0001 C CNN
 F 1 "GND" H 3125 7205 50  0000 C CNN
 F 2 "" H 3125 7355 50  0000 C CNN
@@
 M0/M1/M2:\n0 0 0 - Full Step\n1 0 0 - 1/2 Step\n0 1 0 - 1/4 Step\n1 1 0 - 1/8 Step\n0 0 1 - 1/16 Step\nInternal pull down\n
 $Comp
-L +5V #PWR012
+L +5V #PWR011
 U 1 1 59569A5C
 P 1485 4345
-F 0 "#PWR012" H 1485 4195 50  0001 C CNN
+F 0 "#PWR011" H 1485 4195 50  0001 C CNN
 F 1 "+5V" H 1485 4485 50  0000 C CNN
 F 2 "" H 1485 4345 50  0000 C CNN
@@
 $EndComp
 $Comp
-L GND #PWR013
+L GND #PWR012
 U 1 1 59569A75
 P 5585 2095
-F 0 "#PWR013" H 5585 1845 50  0001 C CNN
+F 0 "#PWR012" H 5585 1845 50  0001 C CNN
 F 1 "GND" H 5585 1945 50  0000 C CNN
 F 2 "" H 5585 2095 50  0000 C CNN
@@
 NoConn ~ 3125 7180
 $Comp
-L GND #PWR014
+L GND #PWR013
 U 1 1 59AC80BA
 P 4270 1110
-F 0 "#PWR014" H 4270 860 50  0001 C CNN
+F 0 "#PWR013" H 4270 860 50  0001 C CNN
 F 1 "GND" H 4270 960 50  0000 C CNN
 F 2 "" H 4270 1110 50  0000 C CNN
@@
 $EndComp
 $Comp
-L +5V #PWR015
+L +5V #PWR014
 U 1 1 59AC8320
 P 4470 1470
-F 0 "#PWR015" H 4470 1320 50  0001 C CNN
+F 0 "#PWR014" H 4470 1320 50  0001 C CNN
 F 1 "+5V" H 4470 1610 50  0000 C CNN
 F 2 "" H 4470 1470 50  0000 C CNN
@@
 $EndComp
 $Comp
-L GND #PWR016
+L GND #PWR015
 U 1 1 59AC848A
 P 2370 1665
-F 0 "#PWR016" H 2370 1415 50  0001 C CNN
+F 0 "#PWR015" H 2370 1415 50  0001 C CNN
 F 1 "GND" H 2370 1515 50  0000 C CNN
 F 2 "" H 2370 1665 50  0000 C CNN
@@
 Connection ~ 1825 4360
 $Comp
-L +5V #PWR017
+L +5V #PWR016
 U 1 1 59ADD131
 P 1450 6490
-F 0 "#PWR017" H 1450 6340 50  0001 C CNN
+F 0 "#PWR016" H 1450 6340 50  0001 C CNN
 F 1 "+5V" H 1450 6630 50  0000 C CNN
 F 2 "" H 1450 6490 50  0000 C CNN
@@
 	1790 6540 1790 6505
 Connection ~ 1790 6505
-Text Notes 4655 5035 0    60   ~ 0
-Blue\nRed\nBlack\nGreen
 Text Notes 4370 7170 0    60   ~ 0
 Green\nBlack\nRed\nBlue
@@
 F 0 "R109" H 5035 1405 50  0000 L CNN
 F 1 "330R" H 5035 1345 50  0000 L CNN
-F 2 "" H 5005 1385 50  0000 C CNN
+F 2 "Resistors_SMD:R_0805_HandSoldering" H 5005 1385 50  0001 C CNN
 F 3 "" H 5005 1385 50  0000 C CNN
 F 4 "Value" H 5005 1385 60  0001 C CNN "Fieldname"
@@
 F 0 "D102" H 4955 1160 50  0000 L CNN
 F 1 "Red LED" H 4830 935 50  0000 L CNN
-F 2 "" V 5005 1035 50  0000 C CNN
+F 2 "LEDs:LED_0805_HandSoldering" V 5005 1035 50  0001 C CNN
 F 3 "" V 5005 1035 50  0000 C CNN
 F 4 "Value" H 5005 1035 60  0001 C CNN "Fieldname"
@@
 $EndComp
 $Comp
-L GND #PWR018
+L GND #PWR017
 U 1 1 5A80ACDE
 P 5005 1545
-F 0 "#PWR018" H 5005 1295 50  0001 C CNN
+F 0 "#PWR017" H 5005 1295 50  0001 C CNN
 F 1 "GND" H 5005 1395 50  0000 C CNN
 F 2 "" H 5005 1545 50  0000 C CNN
@@
 Text Label 1850 1515 0    60   ~ 0
 CE
+Text Notes 4630 5040 0    60   ~ 0
+Green\nBlack\nRed\nBlue
 $EndSCHEMATC

Commit message: changed stepper drivers to A4988 on pcb and schematic
Parts:
- removed U102, U103: DRV8825, balancingBot:DRV8825, symbol DRV8825
- added U102, U103: A4988, balancingBot:A4988, symbol A4988
Connections:
- net +5V: now also U102.11 (~SLP), U102.12 (~RST), U102.7 (VDD), U103.11 (~SLP), U103.12 (~RST), U103.7 (VDD)
- net 11.75V: now also U102.1 (VMOT), U103.1 (VMOT)
- net GND: now also U102.2 (GND), U102.8 (GND), U103.2 (GND), U103.8 (GND)
- net Ldir: now also U103.9 (DIR)
- net Lstep: now also U103.10 (STEP)
- net Rdir: now also U102.9 (DIR)
- net Rstep: now also U102.10 (STEP)
- net at R106.2: now also U102.13 (MS3)
- net at R107.1: now also U102.14 (MS2)
- net at R108.2: now also U102.15 (MS1)
- net at P101.1 (P1): now also U102.3 (2B)
- net at P101.2 (P2): now also U102.4 (2A)
- net at P101.3 (P3): now also U102.5 (1A)
- net at P101.4 (P4): now also U102.6 (1B)
- net at R103.2: now also U103.13 (MS3)
- net at R104.1: now also U103.14 (MS2)
- net at R105.2: now also U103.15 (MS1)
- net at P102.1 (P1): now also U103.3 (2B)
- net at P102.2 (P2): now also U103.4 (2A)
- net at P102.3 (P3): now also U103.5 (1A)
- net at P102.4 (P4): now also U103.6 (1B)
- no-connect marks 24 -> 22
Changed lines of the file:
@@
 $EndDescr
-$Comp
-L DRV8825 U102
-U 1 1 5955942F
-P 2665 6960
-F 0 "U102" H 2655 6510 60  0000 C CNN
-F 1 "DRV8825" H 2665 7370 60  0000 C CNN
-F 2 "balancingBot:DRV8825" H 2665 6960 60  0001 C CNN
-F 3 "" H 2665 6960 60  0001 C CNN
-	1    2665 6960
-	1    0    0    -1
-$EndComp
 $Comp
 L GY-521 U106
@@
 F 3 "" H 1300 1895 60  0001 C CNN
 	1    1300 1895
-	1    0    0    -1
-$EndComp
-$Comp
-L DRV8825 U103
-U 1 1 59559506
-P 2700 4815
-F 0 "U103" H 2690 4365 60  0000 C CNN
-F 1 "DRV8825" H 2700 5225 60  0000 C CNN
-F 2 "balancingBot:DRV8825" H 2700 4815 60  0001 C CNN
-F 3 "" H 2700 4815 60  0001 C CNN
-	1    2700 4815
 	1    0    0    -1
 $EndComp
@@
 NoConn ~ 1850 2145
 NoConn ~ 2240 4585
-NoConn ~ 3160 5035
 Text Label 2240 5035 2    50   ~ 0
 Lstep
@@
 Ldir
 NoConn ~ 2205 6730
-NoConn ~ 3125 7180
 $Comp
 L GND #PWR013
@@
 Text Notes 4630 5040 0    60   ~ 0
 Green\nBlack\nRed\nBlue
+$Comp
+L A4988 U103
+U 1 1 5B39365B
+P 2700 4815
+F 0 "U103" H 2690 4365 60  0000 C CNN
+F 1 "A4988" H 2700 5225 60  0000 C CNN
+F 2 "balancingBot:A4988" H 2700 4815 60  0001 C CNN
+F 3 "" H 2700 4815 60  0001 C CNN
+F 4 "Value" H 2700 4815 60  0001 C CNN "Fieldname"
+	1    2700 4815
+	1    0    0    -1
+$EndComp
+$Comp
+L A4988 U102
+U 1 1 5B3936CD
+P 2665 6960
+F 0 "U102" H 2655 6510 60  0000 C CNN
+F 1 "A4988" H 2665 7370 60  0000 C CNN
+F 2 "balancingBot:A4988" H 2665 6960 60  0001 C CNN
+F 3 "" H 2665 6960 60  0001 C CNN
+F 4 "Value" H 2665 6960 60  0001 C CNN "Fieldname"
+	1    2665 6960
+	1    0    0    -1
+$EndComp
+$Comp
+L +5V #PWR018
+U 1 1 5B394B01
+P 3540 7340
+F 0 "#PWR018" H 3540 7190 50  0001 C CNN
+F 1 "+5V" H 3540 7480 50  0000 C CNN
+F 2 "" H 3540 7340 50  0000 C CNN
+F 3 "" H 3540 7340 50  0000 C CNN
+	1    3540 7340
+	1    0    0    -1
+$EndComp
+Wire Wire Line
+	3125 7180 3370 7180
+Wire Wire Line
+	3370 7180 3370 7340
+Wire Wire Line
+	3370 7340 3540 7340
+$Comp
+L +5V #PWR019
+U 1 1 5B394D24
+P 3510 5195
+F 0 "#PWR019" H 3510 5045 50  0001 C CNN
+F 1 "+5V" H 3510 5335 50  0000 C CNN
+F 2 "" H 3510 5195 50  0000 C CNN
+F 3 "" H 3510 5195 50  0000 C CNN
+	1    3510 5195
+	1    0    0    -1
+$EndComp
+Wire Wire Line
+	3160 5035 3335 5035
+Wire Wire Line
+	3335 5035 3335 5195
+Wire Wire Line
+	3335 5195 3510 5195
 $EndSCHEMATC
